Commit message: kukaa-env

File: my_py_bullet/kuka_env/kuka_env_/envs/agents/assets/iiwa/urdf/iiwa14_rs_scanner_v1.urdf (robot description, URDF)
Before this commit: robot iiwa14_rs_scanner_v1, 12 links, 11 joints
Links:
- link iiwa_link_0: geometry collision mesh filename=meshes/iiwa14/visual/link_0.stl; visual mesh filename=meshes/iiwa14/visual/link_0.stl
- link iiwa_link_1: geometry collision mesh filename=meshes/iiwa14/visual/link_1.stl; visual mesh filename=meshes/iiwa14/visual/link_1.stl
- link iiwa_link_2: geometry collision mesh filename=meshes/iiwa14/visual/link_2.stl; visual mesh filename=meshes/iiwa14/visual/link_2.stl
- link iiwa_link_3: geometry collision mesh filename=meshes/iiwa14/visual/link_3.stl; visual mesh filename=meshes/iiwa14/visual/link_3.stl
- link iiwa_link_4: geometry collision mesh filename=meshes/iiwa14/visual/link_4.stl; visual mesh filename=meshes/iiwa14/visual/link_4.stl
- link iiwa_link_5: geometry collision mesh filename=meshes/iiwa14/visual/link_5.stl; visual mesh filename=meshes/iiwa14/visual/link_5.stl
- link iiwa_link_6: geometry collision mesh filename=meshes/iiwa14/visual/link_6.stl; visual mesh filename=meshes/iiwa14/visual/link_6.stl
- link iiwa_link_7: geometry collision mesh filename=meshes/iiwa14/visual/link_7.stl; visual mesh filename=meshes/iiwa14/visual/link_7.stl
- link tool_link: geometry collision mesh filename=meshes/tools/visual/Scanner_mount_assem_prt.STL; visual mesh filename=meshes/tools/visual/Scanner_mount_assem_prt.STL
