Commit message: apply/check random policy

File: my_py_bullet/kuka_env/kuka_env_example/envs/agents/assets/iiwa/urdf/iiwa14_rs_scanner_v1.urdf (robot description, URDF)
Before this commit: robot iiwa14_rs_scanner_v1, 12 links, 11 joints
Links:
- link tool_link: mass None -> 1.3
- link tool_link_ee: mass None -> 1e-6
